Commit message: fix safe_home

File: urdf/00-arm-rs_asm-v3/urdf/00-arm-rs_asm-v3.urdf (robot description, URDF)
Before this commit: robot 00-arm-rs_asm-v3, 10 links, 9 joints
Links:
- link base_link: mass 0.57955856181278 -> 1.1774
- link gripper_end: mass 0.125579259385149 -> 0.65
- link gripper_left: mass 0.0401440141138942 -> 0.0752
- link gripper_right: mass 0.0401440141138941 -> 0.0752
- link link1: mass 0.153290856769315 -> 0.4655
- link link2: mass 0.753322079867911 -> 1.972
- link link3: mass 0.519938325740626 -> 1.062
- link link4: mass 0.163567538196875 -> 0.66
- link link6: mass 0.0182990324327459 -> 0.03
