Commit message: fix rs urdf link2 mass

File: urdf/00-arm-rs_asm-v3/urdf/00-arm-rs_asm-v3.urdf (robot description, URDF)
Before this commit: robot 00-arm-rs_asm-v3, 10 links, 9 joints
Links:
- link link2: mass 1.972 -> 1.772

Commit message: Update the mass in 00-arm-rs_asm-v3. urdf

File: urdf/00-arm-rs_asm-v3/urdf/00-arm-rs_asm-v3.urdf (robot description, URDF)
Before this commit: robot 00-arm-rs_asm-v3, 10 links, 9 joints
Links:
- link link2: mass 1.772 -> 1.552
- link link3: mass 1.062 -> 1.252
- link link4: mass 0.66 -> 0.46
- link link5: mass 0.150120457182895 -> 0.20120457182895
- link link6: mass 0.03 -> 0.1
