Commit message: rs

File: urdf/reBot-DevArm_fixend_description/urdf/reBot-DevArm_fixend.urdf (robot description, URDF)
Before this commit: robot reBot-DevArm_fixend, 8 links, 7 joints
Links:
- link base_link: geometry collision mesh filename=meshes/base_link.STL; visual mesh filename=meshes/base_link.STL
- link end_link: geometry collision mesh filename=meshes/end_link.STL; visual mesh filename=meshes/end_link.STL
- link link1: geometry collision mesh filename=meshes/link1.STL; visual mesh filename=meshes/link1.STL
- link link2: geometry collision mesh filename=meshes/link2.STL; visual mesh filename=meshes/link2.STL
- link link3: geometry collision mesh filename=meshes/link3.STL; visual mesh filename=meshes/link3.STL
- link link4: geometry collision mesh filename=meshes/link4.STL; visual mesh filename=meshes/link4.STL
- link link5: geometry collision mesh filename=meshes/link5.STL; visual mesh filename=meshes/link5.STL
- link link6: geometry collision mesh filename=meshes/link6.STL; visual mesh filename=meshes/link6.STL
Joints:
- removed joint join3
- added joint joint3: type revolute, parent link2, child link3, origin xyz=-0.264 0 0 rpy=0 0 0, axis 0 0 1, limit lower=-3.14 upper=0 effort=27 velocity=50

Commit message: add EN and fix dm urdf

File: urdf/reBot-DevArm_fixend_description/urdf/reBot-DevArm_fixend.urdf (robot description, URDF)
Before this commit: robot reBot-DevArm_fixend, 8 links, 7 joints
Links:
- link end_link: mass 0.5500000 -> 0.4500000
